File: PCB/portable-hackpad.kicad_pcb (KiCad board)
At the start: 2 copper layers, 7 parts, among them SW1 SW_Push, SW2 SW_Push, SW3 SW_Push, SW4 SW_Push, U1 XIAO-RP2040-DIP

Commit message: define edges
Other:
- board outline added: 42.1 x 63.5 mm
Changed lines of the file:
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@@
 		)
 	)
+	(gr_rect
+		(start 161.4 83.7)
+		(end 203.5 147.2)
+		(stroke
+			(width 0.05)
+			(type default)
+		)
+		(fill none)
+		(layer "Edge.Cuts")
+	)
 )

Commit message: fix edges
Other:
- board size 42.1 x 63.5 mm -> 42.1 x 70 mm
Changed lines of the file:
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@@
 	(gr_rect
 		(start 161.4 83.7)
-		(end 203.5 147.2)
+		(end 203.5 153.7)
 		(stroke
 			(width 0.05)

Commit message: routing
Routing:
- net GND: track 0.00 -> 86.7 mm, vias 0 -> 6
- net Net-(D1-DOUT): track 0.00 -> 52.6 mm, vias 0 -> 2
- net Net-(U1-GPIO4/MISO): track 0.00 -> 49.5 mm, vias 0 -> 1
- net Net-(U1-GPIO3/MOSI): track 0.00 -> 44.4 mm, vias 0 -> 2
- net +5V: track 0.00 -> 40.5 mm
- net Net-(U1-GPIO1/RX): track 0.00 -> 28.5 mm
- net Net-(U1-GPIO2/SCK): track 0.00 -> 18.0 mm, vias 0 -> 2
- net Net-(D1-DIN): track 0.00 -> 6.16 mm

Commit message: add branding
Other:
- board text added: "Lilia's Portable Hackpad"
